File: G_One_PCB/G_One_PCB/G_One_PCB.kicad_pcb (KiCad board)
At the start: 2 copper layers, 219.2 x 133.8 mm, 95 parts, among them K01(ESC)1 KEYSW, K02(F1)1 KEYSW, K03(F2)1 KEYSW, K04(F3)1 KEYSW, K05(F4)1 KEYSW, K07(F5)1 KEYSW, K10(M0)1 KEYSW, K11(_`_)1 KEYSW, K12(1!)1 KEYSW, K13(2@)1 KEYSW, K14(3#)1 KEYSW, K15(4$)1 KEYSW, K16(5%)1 KEYSW, K17(6^)1 KEYSW, K20(M1)1 KEYSW, K21(Tap)1 KEYSW, K22(Q)1 KEYSW, K23(W)1 KEYSW, K24(E)1 KEYSW, K25(R)1 KEYSW, K26(T)1 KEYSW, K27(P)1 KEYSW, K28(IoT0)1 KEYSW, K30(M2)1 KEYSW, K31(Caps_Lock)1 KEYSW, K32(A)1 KEYSW, K33(S)1 KEYSW, K34(D)1 KEYSW, K35(F)1 KEYSW, K36(G)1 KEYSW, K37(H)1 KEYSW, K38(IoT1)1 KEYSW, K40(M3)1 KEYSW, K41(L_Shift)1 KEYSW, K42(Z)1 KEYSW, K43(X)1 KEYSW, K44(C)1 KEYSW, K45(V)1 KEYSW, K46(B)1 KEYSW, K48(IoT2)1 KEYSW, K50(M4)1 KEYSW, K51(L_CTRL)1 KEYSW, K52(Win)1 KEYSW, K53(L_ALT)1 KEYSW, K54(Space)1 KEYSW

Commit message: PCB 기판에 SW 배치 완료(위치 수정 필요)
Parts:
- moved K50(M4)1 464.8 mm to (249.8, 136.5)
- moved K40(M3)1 443.0 mm to (249.8, 117.5)
- moved K41(L_Shift)1 425.9 mm to (209.3, 117.5)
- moved K31(Caps_Lock)1 425.9 mm to (214.1, 98.5)
- moved K21(Tap)1 425.2 mm to (216.5, 79.5)
- moved K52(Win)1 411.6 mm to (195.1, 136.5)
- moved K30(M2)1 401.9 mm to (249.8, 98.5)
- moved K51(L_CTRL)1 389.6 mm to (218.9, 136.5)
- moved D1 382.5 mm to (221.0, 50.4)
- moved K54(Space)1 364.6 mm to (133.4, 136.5)
- moved K53(L_ALT)1 358.7 mm to (171.5, 136.5)
- moved K43(X)1 350.4 mm to (159.5, 117.5)
- moved K33(S)1 341.1 mm to (169.0, 98.5)
- moved K20(M1)1 337.8 mm to (249.8, 79.5)
- moved K01(ESC)1 324.2 mm to (221.2, 36.8)
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Other:
- outline, holes or cut-outs redrawn

Commit message: G.One 키보드 PCB 디자인 완료 / 거버 파일 생성
Parts:
- removed LeftBottom, LeftTop, RightBottom, RightTop: 3.2mm_M3, MountingHole:MountingHole_3.2mm_M3_ISO7380
- moved D7 326.7 mm to (169.0, -116.8), turned to 90 degrees
- moved D44 323.5 mm to (135.8, -36.0), turned to 90 degrees
- moved D48 322.2 mm to (211.8, -17.0), turned to 90 degrees
- moved D38 318.5 mm to (211.8, -36.0), turned to 90 degrees
- moved D46 291.5 mm to (173.8, -36.0), turned to 90 degrees
- moved D28 290.8 mm to (211.8, -55.0), turned to 90 degrees
- moved K10(M0)1 278.8 mm to (17.0, -93.0)
- moved K20(M1)1 278.8 mm to (17.0, -74.0)
- moved K30(M2)1 278.8 mm to (17.0, -55.0)
- moved K40(M3)1 278.8 mm to (17.0, -36.0)
- moved K50(M4)1 278.8 mm to (17.0, -17.0)
- moved D4 278.7 mm to (121.5, -116.8), turned to 90 degrees
- moved D37 274.1 mm to (183.2, -55.0), turned to 90 degrees
- moved D45 272.5 mm to (154.8, -36.0), turned to 90 degrees
- moved D15 267.4 mm to (131.0, -93.0), turned to 90 degrees
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Routing:
- net /col1: track 0.00 -> 289.9 mm, vias 0 -> 4
- net /col2: track 0.00 -> 278.4 mm, vias 0 -> 4
- net /row4: track 0.00 -> 270.9 mm
- net /row5: track 0.00 -> 263.5 mm
- net /col0: track 0.00 -> 262.2 mm, vias 0 -> 2
- net /row3: track 0.00 -> 256.4 mm
- net /col3: track 0.00 -> 255.5 mm, vias 0 -> 4
- net /row2: track 0.00 -> 236.9 mm
- net /col4: track 0.00 -> 235.0 mm, vias 0 -> 4
- net /row1: track 0.00 -> 204.3 mm
- net /col5: track 0.00 -> 193.6 mm, vias 0 -> 4
- net /row0: track 0.00 -> 171.7 mm
- net /col6: track 0.00 -> 140.3 mm, vias 0 -> 2
- net /col7: track 0.00 -> 95.2 mm
- net /col8: track 0.00 -> 52.0 mm
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Other:
- board outline removed
