File: G_One_PCB/G_One_PCB/G_One_PCB.sch (KiCad schematic (older format))
At the start: 91 parts, among them K01(ESC)1 KEYSW, K02(F1)1 KEYSW, K03(F2)1 KEYSW, K04(F3)1 KEYSW, K05(F4)1 KEYSW, K07(F5)1 KEYSW, K10(M0)1 KEYSW, K11(_`_)1 KEYSW, K12(1!)1 KEYSW, K13(2@)1 KEYSW, K14(3#)1 KEYSW, K15(4$)1 KEYSW, K16(5%)1 KEYSW, K17(6^)1 KEYSW, K20(M1)1 KEYSW, K21(Tap)1 KEYSW, K22(Q)1 KEYSW, K23(W)1 KEYSW, K24(E)1 KEYSW, K25(R)1 KEYSW, K26(T)1 KEYSW, K27(P)1 KEYSW, K28(IoT0)1 KEYSW, K30(M2)1 KEYSW, K31(Caps_Lock)1 KEYSW, K32(A)1 KEYSW, K33(S)1 KEYSW, K34(D)1 KEYSW, K35(F)1 KEYSW, K36(G)1 KEYSW, K37(H)1 KEYSW, K38(IoT1)1 KEYSW, K40(M3)1 KEYSW, K41(L_Shift)1 KEYSW, K42(Z)1 KEYSW, K43(X)1 KEYSW, K44(C)1 KEYSW, K45(V)1 KEYSW, K46(B)1 KEYSW, K48(IoT2)1 KEYSW, K50(M4)1 KEYSW, K51(L_CTRL)1 KEYSW, K52(Win)1 KEYSW, K53(L_ALT)1 KEYSW, K54(Space)1 KEYSW

Commit message: G.One 키보드 PCB 디자인 완료 / 거버 파일 생성
Parts:
- B0: symbol SparkFun-Boards:SPARKFUN_PRO_MICRO -> G_One_PCB-rescue:SPARKFUN_PRO_MICRO-SparkFun-Boards
- D1, D10, D11, D12, D13, D14, D15, D16, D17, D2, D20, D21, D22, D23, D24, D25, D26, D27, D28, D3, D30, D31, D32, D33, D34, D35, D36, D37, D38, D4, D40, D41, D42, D43, D44, D45, D46, D48, D5, D50, D51, D52, D53, D54, D7: symbol keyboard_parts:D -> G_One_PCB-rescue:D-keyboard_parts
- K01(ESC)1, K02(F1)1, K03(F2)1, K04(F3)1, K05(F4)1, K07(F5)1, K10(M0)1, K11(_`_)1, K12(1!)1, K13(2@)1, K14(3#)1, K15(4$)1, K16(5%)1, K17(6^)1, K20(M1)1, K21(Tap)1, K22(Q)1, K23(W)1, K24(E)1, K25(R)1, K26(T)1, K27(P)1, K28(IoT0)1, K30(M2)1, K31(Caps_Lock)1, K32(A)1, K33(S)1, K34(D)1, K35(F)1, K36(G)1, K37(H)1, K38(IoT1)1, K40(M3)1, K41(L_Shift)1, K42(Z)1, K43(X)1, K44(C)1, K45(V)1, K46(B)1, K48(IoT2)1, K50(M4)1, K51(L_CTRL)1, K52(Win)1, K53(L_ALT)1, K54(Space)1: symbol keyboard_parts:KEYSW -> G_One_PCB-rescue:KEYSW-keyboard_parts
